File: hardware/bubble.kicad_pcb (KiCad board)
At the start: 4 copper layers, 100 x 100 mm, 56 parts, among them J1 Barrel_Jack_Switch, Q1 AO3400A, U1 i7220, U2 i7230, U3 i7254, U4 i7250, U5 i7254, U6 i7242, U7 LM7805_TO220

Commit message: hardware: new board schematic
Parts:
- removed A1: Arduino_Nano_v3.x, Module:Arduino_Nano
- removed C1, C11, C13, C15, C16, C17, C2, C21, C3, C9: 100nF, Capacitor_SMD:C_0603_1608Metric
- removed C10, C12, C14, C18, C22, C4, C5, C6, C7, C8: 22uF, Capacitor_SMD:C_1206_3216Metric
- removed C19, C20: 120pF, Capacitor_SMD:C_0603_1608Metric
- removed C23: 1uF, Capacitor_SMD:C_0603_1608Metric
- removed C24: 2.2uF, Capacitor_SMD:C_0603_1608Metric
- removed C25, C26: 1000uF, Capacitor_THT:CP_Radial_D8.0mm_P5.00mm
- removed J1: Barrel_Jack_Switch, Connector_BarrelJack:BarrelJack_GCT_DCJ200-10-A_Horizontal
- removed JP1, JP2: ~, Connector_PinSocket_2.54mm:PinSocket_1x02_P2.54mm_Vertical
- removed L1, L2, L3: .22uH, Inductor_SMD:L_1008_2520Metric
- removed MBM1: i7110, intel_bubble:MBM_dual
- removed Q1: AO3400A, Package_TO_SOT_SMD:SOT-23
- removed R1, R3, R5: 5.6k, Resistor_SMD:R_0603_1608Metric
- removed R10, R11, R8, R9: 1k 2W, Resistor_SMD:R_2512_6332Metric
- removed R12, R6: 5.1, Resistor_SMD:R_0805_2012Metric
- removed R13: 33k, Resistor_SMD:R_0603_1608Metric
- removed R14: 12k, Resistor_SMD:R_0603_1608Metric
- removed R2: 3.48k 1%, Resistor_SMD:R_0603_1608Metric
- removed R4: 47, Resistor_SMD:R_0805_2012Metric
- removed R7: 10, Resistor_SMD:R_0603_1608Metric
- removed U1: i7220, Package_DIP:DIP-40_W15.24mm
- removed U2: i7230, Package_DIP:DIP-22_W7.62mm
- removed U3, U5: i7254, Package_DIP:DIP-14_W7.62mm
- removed U4: i7250, Package_DIP:DIP-16_W7.62mm
- removed U6: i7242, Package_DIP:DIP-20_W7.62mm
- removed U7: LM7805_TO220, Package_TO_SOT_THT:TO-220-3_Vertical
Routing:
- net +12V: track 298.9 -> 0.00 mm
- net /SYS_~{CS}: track 241.1 -> 0.00 mm
- net /~{RESET.OUT}: track 229.6 -> 0.00 mm, vias 2 -> 0
- net /~{DATA.B}: track 177.1 -> 0.00 mm
- net /~{DATA.A}: track 174.9 -> 0.00 mm
- net +5V: track 147.5 -> 0.00 mm
- net /SWAP: track 129.7 -> 0.00 mm
- net /~{SYNC}: track 110.5 -> 0.00 mm
- net /DIO: track 108.7 -> 0.00 mm
- net /~{SHIFT.CLK}: track 108.0 -> 0.00 mm
- net /~{ERR.FLG}: track 96.8 -> 0.00 mm
- net /CLK: track 88.8 -> 0.00 mm
- net /C/~{D}: track 86.0 -> 0.00 mm
- net /~{PWR.FAIL}: track 76.8 -> 0.00 mm, vias 1 -> 0
- net /A0: track 71.7 -> 0.00 mm
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- removed copper zone on B.Cu, net GND
- removed copper zone on F.Cu, net GND
- removed copper zone on F.Cu, net Net-(C2-Pad1)
- removed copper zone on F.Cu, net Net-(U2-VCC)
Other:
- board outline removed
- board text removed: "2024 grm"
- board text removed: "BOOT SWAP"
- board text removed: "Bubble Def*cker"
- board text removed: "REMOVE JUMPER IF USING 7110AZ"
- board text removed: "UHF"

Commit message: hardware: add powerfail circuit, rework power
Parts:
- added 20pF1: C, Capacitor_SMD:C_0805_2012Metric_Pad1.18x1.45mm_HandSolder, F.Cu at (95.8, 38.5)
- added C1: 0.33 uF, Capacitor_THT:C_Rect_L13.0mm_W6.5mm_P7.50mm_P10.00mm, F.Cu at (95.6, 71.8)
- added C10: 47uF, Capacitor_THT:CP_Radial_D5.0mm_P2.00mm, F.Cu at (79.2, 100.8)
- added C11: 47uF, Capacitor_THT:CP_Radial_D5.0mm_P2.00mm, F.Cu at (79.2, 107.3)
- added C12: 22uF, Capacitor_THT:CP_Radial_D5.0mm_P2.00mm, F.Cu at (85.9, 87.7)
- added C13: 0.1uF, Capacitor_SMD:C_0805_2012Metric_Pad1.18x1.45mm_HandSolder, F.Cu at (95.8, 53.6)
- added C14: 0.1uF, Capacitor_SMD:C_0805_2012Metric_Pad1.18x1.45mm_HandSolder, F.Cu at (100.6, 38.5)
- added C15: 22uF, Capacitor_THT:CP_Radial_D5.0mm_P2.00mm, F.Cu at (85.9, 94.2)
- added C16: 22uF 25V, Capacitor_THT:CP_Radial_D5.0mm_P2.00mm, F.Cu at (85.9, 100.8)
- added C17: 120 pF 100V 5%, Capacitor_THT:C_Disc_D5.0mm_W2.5mm_P2.50mm, F.Cu at (95.4, 77.8)
- added C18: 120 pF 100V 5%, Capacitor_THT:C_Disc_D5.0mm_W2.5mm_P2.50mm, F.Cu at (95.4, 81.9)
- added C19: 0.1uF, Capacitor_SMD:C_0805_2012Metric_Pad1.18x1.45mm_HandSolder, F.Cu at (100.6, 41.6)
- added C2: 22uF, Capacitor_THT:CP_Radial_D4.0mm_P1.50mm, F.Cu at (114.7, 50.3)
- added C20: 0.1uF, Capacitor_SMD:C_0805_2012Metric_Pad1.18x1.45mm_HandSolder, F.Cu at (100.6, 44.6)
- added C21: 0.1uF, Capacitor_SMD:C_0805_2012Metric_Pad1.18x1.45mm_HandSolder, F.Cu at (100.6, 47.6)
- added C22: 22uF, Capacitor_THT:CP_Radial_D5.0mm_P2.00mm, F.Cu at (85.9, 107.3)
- added C23: 2.2 uF, Capacitor_SMD:C_0805_2012Metric_Pad1.18x1.45mm_HandSolder, F.Cu at (100.6, 50.6)
- added C24: 22uF, Capacitor_THT:CP_Radial_D5.0mm_P2.00mm, F.Cu at (92.5, 87.7)
- added C25: 22uF, Capacitor_THT:CP_Radial_D5.0mm_P2.00mm, F.Cu at (92.5, 94.2)
- added C26: 0.01 uF, Capacitor_SMD:C_0805_2012Metric_Pad1.18x1.45mm_HandSolder, F.Cu at (100.6, 53.6)
- added C27: 0.01 uF, Capacitor_SMD:C_0805_2012Metric_Pad1.18x1.45mm_HandSolder, F.Cu at (105.4, 38.5)
- added C28: 10 uF, Capacitor_SMD:C_0805_2012Metric_Pad1.18x1.45mm_HandSolder, F.Cu at (105.4, 41.6)
- added C29: 20pF, Capacitor_SMD:C_0805_2012Metric_Pad1.18x1.45mm_HandSolder, F.Cu at (105.4, 44.6)
- added C3: 47uF, Capacitor_THT:CP_Radial_D5.0mm_P2.00mm, F.Cu at (79.2, 87.7)
- added C30: 22uF, Capacitor_SMD:C_0805_2012Metric_Pad1.18x1.45mm_HandSolder, F.Cu at (105.4, 47.6)
- added C31: 0.1uF, Capacitor_SMD:C_0805_2012Metric_Pad1.18x1.45mm_HandSolder, F.Cu at (105.4, 50.6)
- added C32: 0.1uF, Capacitor_SMD:C_0805_2012Metric_Pad1.18x1.45mm_HandSolder, F.Cu at (105.4, 53.6)
- added C33: 0.1uF, Capacitor_SMD:C_0805_2012Metric_Pad1.18x1.45mm_HandSolder, F.Cu at (110.2, 38.5)
- added C34: 22uF, Capacitor_SMD:C_0805_2012Metric_Pad1.18x1.45mm_HandSolder, F.Cu at (110.2, 41.6)
- added C35: 0.1uF, Capacitor_SMD:C_0805_2012Metric_Pad1.18x1.45mm_HandSolder, F.Cu at (110.2, 44.6)
- added C36: 47uF, Capacitor_THT:CP_Radial_D5.0mm_P2.00mm, F.Cu at (92.5, 100.8)
- added C37: 0.1uF, Capacitor_SMD:C_0805_2012Metric_Pad1.18x1.45mm_HandSolder, F.Cu at (110.2, 47.6)
- added C38: 150uF, Capacitor_THT:CP_Radial_D10.0mm_P2.50mm, F.Cu at (81.6, 127.9)
- added C4: 150uF, Capacitor_THT:CP_Radial_D10.0mm_P2.50mm, F.Cu at (81.6, 116.4)
- added C5: 0.1uF, Capacitor_SMD:C_0805_2012Metric_Pad1.18x1.45mm_HandSolder, F.Cu at (95.8, 41.6)
- added C6: 0.1uF, Capacitor_SMD:C_0805_2012Metric_Pad1.18x1.45mm_HandSolder, F.Cu at (95.8, 44.6)
- added C7: 0.1uF, Capacitor_SMD:C_0805_2012Metric_Pad1.18x1.45mm_HandSolder, F.Cu at (95.8, 47.6)
- added C8: 47uF, Capacitor_THT:CP_Radial_D5.0mm_P2.00mm, F.Cu at (79.2, 94.2)
- added C9: 0.1uF, Capacitor_SMD:C_0805_2012Metric_Pad1.18x1.45mm_HandSolder, F.Cu at (95.8, 50.6)
- added D1: POWER FAILED LED, LED_SMD:LED_0805_2012Metric_Pad1.15x1.40mm_HandSolder, F.Cu at (120.5, 131.3)
- added D2: D, Diode_SMD:D_SOD-323_HandSoldering, F.Cu at (91.2, 132.3)
- added D3: D, Diode_SMD:D_SOD-323_HandSoldering, F.Cu at (91.2, 135.3)
- added D4: LED, LED_SMD:LED_0805_2012Metric_Pad1.15x1.40mm_HandSolder, F.Cu at (120.5, 134.3)
- added J1: Conn_01x03_Pin, Connector_PinHeader_2.54mm:PinHeader_1x03_P2.54mm_Vertical, F.Cu at (120.6, 112.7)
- added J2: Conn_01x04_Pin, Connector_PinHeader_2.54mm:PinHeader_1x04_P2.54mm_Horizontal, F.Cu at (112.7, 57.4)
- added J3: USB-C, Connector_USB:USB_C_Receptacle_HRO_TYPE-C-31-M-12, F.Cu at (118.5, 42.8)
- added J4: 12V Power, Connector_BarrelJack:BarrelJack_Horizontal, F.Cu at (107.9, 60.5)
- added JP1: Only for reseed, Connector_PinHeader_2.54mm:PinHeader_1x02_P2.54mm_Vertical, F.Cu at (102.2, 78.1)
- added L1: 0.22 uH, Inductor_SMD:L_APV_APH0530, F.Cu at (92.4, 114.0)
- added L2: 0.22 uH, Inductor_SMD:L_APV_APH0530, F.Cu at (92.4, 120.7)
- added L3: 0.22 uH, Inductor_SMD:L_APV_APH0530, F.Cu at (92.4, 127.5)
- added MBM1: i7110, intel_bubble:MBM_socket, F.Cu at (62.8, 60.7)
- added Q1: BS170, Package_TO_SOT_THT:TO-92_Inline, F.Cu at (68.1, 133.3)
- added Q2: DTC113Z, Package_TO_SOT_SMD:SOT-23-3, F.Cu at (120.8, 49.7)
- added R1: 5.1k, Resistor_SMD:R_0805_2012Metric_Pad1.20x1.40mm_HandSolder, F.Cu at (109.9, 90.0)
- added R10: 33k, Resistor_SMD:R_0805_2012Metric_Pad1.20x1.40mm_HandSolder, F.Cu at (114.7, 95.9)
- added R11: 5.1, Resistor_SMD:R_0805_2012Metric_Pad1.20x1.40mm_HandSolder, F.Cu at (114.7, 98.9)
- added R12: 5.1, Resistor_SMD:R_0805_2012Metric_Pad1.20x1.40mm_HandSolder, F.Cu at (114.7, 101.8)
- added R13: 5.1k, Resistor_SMD:R_0805_2012Metric_Pad1.20x1.40mm_HandSolder, F.Cu at (114.7, 104.8)
- added R14: 300Ohm, Resistor_SMD:R_0805_2012Metric_Pad1.20x1.40mm_HandSolder, F.Cu at (114.7, 107.7)
- added R15: 5.1k, Resistor_SMD:R_0805_2012Metric_Pad1.20x1.40mm_HandSolder, F.Cu at (119.4, 90.0)
- added R16: 5.1k, Resistor_SMD:R_0805_2012Metric_Pad1.20x1.40mm_HandSolder, F.Cu at (119.4, 93.0)
- added R17: 22, Resistor_SMD:R_0805_2012Metric_Pad1.20x1.40mm_HandSolder, F.Cu at (119.4, 95.9)
- added R18: 22, Resistor_SMD:R_0805_2012Metric_Pad1.20x1.40mm_HandSolder, F.Cu at (119.4, 98.9)
- added R19: 1.5k, Resistor_SMD:R_0805_2012Metric_Pad1.20x1.40mm_HandSolder, F.Cu at (119.4, 101.8)
- added R2: 5.1k, Resistor_SMD:R_0805_2012Metric_Pad1.20x1.40mm_HandSolder, F.Cu at (109.9, 93.0)
- added R3: 3.48k, Resistor_SMD:R_0805_2012Metric_Pad1.20x1.40mm_HandSolder, F.Cu at (109.9, 95.9)
- added R4: 10, Resistor_SMD:R_0805_2012Metric_Pad1.20x1.40mm_HandSolder, F.Cu at (109.9, 98.9)
- added R5: 300, Resistor_SMD:R_0805_2012Metric_Pad1.20x1.40mm_HandSolder, F.Cu at (109.9, 101.8)
- added R6: 47, Resistor_SMD:R_0805_2012Metric_Pad1.20x1.40mm_HandSolder, F.Cu at (109.9, 104.8)
- added R7: 1k, Resistor_SMD:R_0805_2012Metric_Pad1.20x1.40mm_HandSolder, F.Cu at (109.9, 107.7)
- added R8: 3.9k, Resistor_SMD:R_0805_2012Metric_Pad1.20x1.40mm_HandSolder, F.Cu at (114.7, 90.0)
- added R9: 5.5k, Resistor_SMD:R_0805_2012Metric_Pad1.20x1.40mm_HandSolder, F.Cu at (114.7, 93.0)
- added RN1: 1k, Resistor_THT:R_Array_SIP8, F.Cu at (98.9, 86.5)
- added SW1: Reset, Button_Switch_THT:SW_PUSH_6mm_H5mm, F.Cu at (54.8, 127.3)
- added U1: 74LS74, Package_SO:SOIC-14_3.9x8.7mm_P1.27mm, F.Cu at (70.3, 116.6)
- added U10: STM32F103C8Tx, Package_QFP:LQFP-48_7x7mm_P0.5mm, F.Cu at (58.4, 119.6)
- added U11: AMS1117-3.3, Package_TO_SOT_SMD:SOT-223-3_TabPin2, F.Cu at (71.0, 125.9)
- added U2: i7220, Package_DIP:DIP-40_W15.24mm, F.Cu at (36.0, 86.4)
- added U3: i7242, Package_DIP:DIP-20_W7.62mm, F.Cu at (67.7, 86.4)
- added U4: i7250, Package_DIP:DIP-16_W7.62mm, F.Cu at (98.4, 90.6)
- added U5: i7230, Package_DIP:DIP-22_W10.16mm, F.Cu at (54.3, 86.4)
- added U6: 74AHC1G00, Package_TO_SOT_SMD:SOT-23-5_HandSoldering, F.Cu at (121.2, 122.5)
- added U7: i7254, Package_DIP:DIP-14_W7.62mm, F.Cu at (98.4, 112.5)
- added U8: i7254, Package_DIP:DIP-14_W7.62mm, F.Cu at (109.1, 112.5)
- added U9: 74LVC1G07, Package_TO_SOT_SMD:SOT-23-5_HandSoldering, F.Cu at (121.2, 127.3)
- added Y1: 8.000 MHz, Oscillator:Oscillator_DIP-8, F.Cu at (111.2, 78.7)
- added Y2: 8Mhz, Crystal:Crystal_SMD_HC49-SD_HandSoldering, F.Cu at (107.5, 133.2)
