File: hardware/bubble.kicad_sch (KiCad schematic)
At the start: 62 parts, among them Q1 BS170, Q2 DTC113Z, U1 74LS74, U2 i7220, U3 i7242, U4 i7250, U5 i7230, U6 74AHC1G00, U7 i7254, U8 i7254, U9 74LVC1G07, Y1 8.000 MHz

Commit message: hardware: connect input signals from 7220 to stm32 five tolerant pins
Connections:
- net CLK renamed MBM CLK
- net ~{BUS.RD}: no longer names the net of U2.25 (~{BUS.RD})
- net ~{RESET.BUS} renamed ~{RESET}
- no-connect marks 9 -> 10
Changed lines of the file:
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@@
 	)
 	(no_connect
+		(at 209.55 276.86)
+	)
+	(no_connect
 		(at 186.69 52.07)
 	)
@@
 	)
 	(global_label "~{WAIT}"
-		(shape input)
+		(shape bidirectional)
 		(at 209.55 274.32 0)
 		(fields_autoplaced yes)
@@
 		)
 		(property "Intersheetrefs" "${INTERSHEET_REFS}"
-			(at 216.6476 274.32 0)
+			(at 217.7589 274.32 0)
 			(hide yes)
 			(show_name no)
@@
 		)
 	)
-	(global_label "~{RESET.BUS}"
+	(global_label "~{RESET}"
 		(shape input)
-		(at 307.34 189.23 180)
+		(at 302.26 311.15 180)
 		(fields_autoplaced yes)
 		(effects
@@
 		)
 		(property "Intersheetrefs" "${INTERSHEET_REFS}"
-			(at 294.1949 189.23 0)
+			(at 293.5297 311.15 0)
 			(hide yes)
 			(show_name no)
@@
 		)
 	)
-	(global_label "CLK"
+	(global_label "MBM CLK"
 		(shape input)
 		(at 175.26 287.02 180)
@@
 		)
 		(property "Intersheetrefs" "${INTERSHEET_REFS}"
-			(at 168.7067 287.02 0)
+			(at 163.5663 287.02 0)
 			(hide yes)
 			(show_name no)
@@
 	)
 	(global_label "D7"
-		(shape input)
+		(shape bidirectional)
 		(at 175.26 269.24 180)
 		(fields_autoplaced yes)
@@
 		)
 		(property "Intersheetrefs" "${INTERSHEET_REFS}"
-			(at 169.7953 269.24 0)
+			(at 168.684 269.24 0)
 			(hide yes)
 			(show_name no)
@@
 	)
 	(global_label "D3"
-		(shape input)
+		(shape bidirectional)
 		(at 175.26 259.08 180)
 		(fields_autoplaced yes)
@@
 		)
 		(property "Intersheetrefs" "${INTERSHEET_REFS}"
-			(at 169.7953 259.08 0)
+			(at 168.684 259.08 0)
 			(hide yes)
 			(show_name no)
@@
 	)
 	(global_label "D0"
-		(shape input)
+		(shape bidirectional)
 		(at 175.26 251.46 180)
 		(fields_autoplaced yes)
@@
 		)
 		(property "Intersheetrefs" "${INTERSHEET_REFS}"
-			(at 169.7953 251.46 0)
+			(at 168.684 251.46 0)
 			(hide yes)
 			(show_name no)
@@
 	)
 	(global_label "INT"
-		(shape input)
+		(shape output)
 		(at 175.26 276.86 180)
 		(fields_autoplaced yes)
@@
 	)
 	(global_label "~{DET.ON}"
-		(shape input)
+		(shape output)
 		(at 175.26 274.32 180)
 		(fields_autoplaced yes)
@@
 		)
 	)
-	(global_label "D4"
+	(global_label "~{RESET}"
 		(shape input)
+		(at 307.34 189.23 180)
+		(fields_autoplaced yes)
+		(effects
+			(font
+				(size 1.27 1.27)
+			)
+			(justify right)
+		)
+		(property "Intersheetrefs" "${INTERSHEET_REFS}"
+			(at 298.6097 189.23 0)
+			(hide yes)
+			(show_name no)
+			(do_not_autoplace no)
+			(effects
+				(font
+					(size 1.27 1.27)
+				)
+				(justify right)
+			)
+		)
+	)
+	(global_label "D4"
+		(shape bidirectional)
 		(at 175.26 261.62 180)
 		(fields_autoplaced yes)
@@
 		)
 		(property "Intersheetrefs" "${INTERSHEET_REFS}"
-			(at 169.7953 261.62 0)
+			(at 168.684 261.62 0)
 			(hide yes)
 			(show_name no)
@@
 	)
 	(global_label "D8"
-		(shape input)
+		(shape bidirectional)
 		(at 175.26 271.78 180)
 		(fields_autoplaced yes)
@@
 		)
 		(property "Intersheetrefs" "${INTERSHEET_REFS}"
-			(at 169.7953 271.78 0)
+			(at 168.684 271.78 0)
 			(hide yes)
 			(show_name no)
@@
 	)
 	(global_label "D6"
-		(shape input)
+		(shape bidirectional)
 		(at 175.26 266.7 180)
 		(fields_autoplaced yes)
@@
 		)
 		(property "Intersheetrefs" "${INTERSHEET_REFS}"
-			(at 169.7953 266.7 0)
+			(at 168.684 266.7 0)
 			(hide yes)
 			(show_name no)
@@
 	)
 	(global_label "~{DACK}"
-		(shape input)
+		(shape output)
 		(at 175.26 246.38 180)
 		(fields_autoplaced yes)
@@
 	)
 	(global_label "D5"
-		(shape input)
+		(shape bidirectional)
 		(at 175.26 264.16 180)
 		(fields_autoplaced yes)
@@
 		)
 		(property "Intersheetrefs" "${INTERSHEET_REFS}"
-			(at 169.7953 264.16 0)
+			(at 168.684 264.16 0)
 			(hide yes)
 			(show_name no)
@@
 		)
 	)
-	(global_label "CLK"
-		(shape input)
+	(global_label "MBM CLK"
+		(shape output)
 		(at 154.94 52.07 0)
 		(fields_autoplaced yes)
@@
 		)
 		(property "Intersheetrefs" "${INTERSHEET_REFS}"
-			(at 161.4933 52.07 0)
+			(at 166.6337 52.07 0)
 			(hide yes)
 			(show_name no)
@@
 		)
 	)
-	(global_label "~{ERR_FLAG}"
+	(global_label "~{RESET}"
 		(shape input)
-		(at 175.26 284.48 180)
+		(at 302.26 219.71 180)
 		(fields_autoplaced yes)
 		(effects
@@
 		)
 		(property "Intersheetrefs" "${INTERSHEET_REFS}"
-			(at 163.1429 284.48 0)
+			(at 293.5297 219.71 0)
 			(hide yes)
 			(show_name no)
@@
 		)
 	)
-	(global_label "~{RESET.BUS}"
-		(shape input)
-		(at 458.47 116.84 0)
-		(fields_autoplaced yes)
-		(effects
-			(font
-				(size 1.27 1.27)
-			)
-			(justify left)
-		)
-		(property "Intersheetrefs" "${INTERSHEET_REFS}"
-			(at 471.6151 116.84 0)
-			(hide yes)
-			(show_name no)
-			(do_not_autoplace no)
-			(effects
-				(font
-					(size 1.27 1.27)
-				)
-				(justify left)
-			)
-		)
-	)
-	(global_label "~{CS}"
-		(shape input)
-		(at 175.26 279.4 180)
+	(global_label "~{ERR_FLAG}"
+		(shape output)
+		(at 175.26 284.48 180)
 		(fields_autoplaced yes)
 		(effects
@@
 		)
 		(property "Intersheetrefs" "${INTERSHEET_REFS}"
-			(at 169.7953 279.4 0)
+			(at 163.1429 284.48 0)
 			(hide yes)
 			(show_name no)
@@
 		)
 	)
-	(global_label "D1"
-		(shape input)
-		(at 175.26 254 180)
+	(global_label "~{RESET}"
+		(shape output)
+		(at 458.47 116.84 0)
 		(fields_autoplaced yes)
 		(effects
@@
 				(size 1.27 1.27)
 			)
-			(justify right)
+			(justify left)
 		)
 		(property "Intersheetrefs" "${INTERSHEET_REFS}"
-			(at 169.7953 254 0)
+			(at 467.2003 116.84 0)
 			(hide yes)
 			(show_name no)
@@
 					(size 1.27 1.27)
 				)
-				(justify right)
+				(justify left)
 			)
 		)
 	)
-	(global_label "~{WR}"
+	(global_label "~{CS}"
 		(shape input)
-		(at 175.26 243.84 180)
+		(at 175.26 279.4 180)
 		(fields_autoplaced yes)
 		(effects
@@
 		)
 		(property "Intersheetrefs" "${INTERSHEET_REFS}"
-			(at 169.5534 243.84 0)
+			(at 169.7953 279.4 0)
 			(hide yes)
 			(show_name no)
@@
 		)
 	)
-	(global_label "~{RESET.BUS}"
-		(shape input)
-		(at 302.26 219.71 180)
+	(global_label "D1"
+		(shape bidirectional)
+		(at 175.26 254 180)
 		(fields_autoplaced yes)
 		(effects
@@
 		)
 		(property "Intersheetrefs" "${INTERSHEET_REFS}"
-			(at 289.1149 219.71 0)
+			(at 168.684 254 0)
 			(hide yes)
 			(show_name no)
@@
 		)
 	)
-	(global_label "~{BUS.RD}"
+	(global_label "~{WR}"
 		(shape input)
-		(at 209.55 276.86 0)
+		(at 175.26 243.84 180)
 		(fields_autoplaced yes)
 		(effects
@@
 				(size 1.27 1.27)
 			)
-			(justify left)
+			(justify right)
 		)
 		(property "Intersheetrefs" "${INTERSHEET_REFS}"
-			(at 219.49 276.86 0)
+			(at 169.5534 243.84 0)
 			(hide yes)
 			(show_name no)
@@
 					(size 1.27 1.27)
 				)
-				(justify left)
+				(justify right)
 			)
 		)
@@
 		)
 	)
-	(global_label "~{RESET.BUS}"
-		(shape input)
-		(at 302.26 311.15 180)
-		(fields_autoplaced yes)
-		(effects
-			(font
-				(size 1.27 1.27)
-			)
-			(justify right)
-		)
-		(property "Intersheetrefs" "${INTERSHEET_REFS}"
-			(at 289.1149 311.15 0)
-			(hide yes)
-			(show_name no)
-			(do_not_autoplace no)
-			(effects
-				(font
-					(size 1.27 1.27)
-				)
-				(justify right)
-			)
-		)
-	)
 	(global_label "D2"
-		(shape input)
+		(shape bidirectional)
 		(at 175.26 256.54 180)
 		(fields_autoplaced yes)
@@
 		)
 		(property "Intersheetrefs" "${INTERSHEET_REFS}"
-			(at 169.7953 256.54 0)
+			(at 168.684 256.54 0)
 			(hide yes)
 			(show_name no)
